File: crossover/crossover.kicad_pcb (KiCad board)
At the start: 2 copper layers, 100 x 84 mm, 18 parts, among them J1 IN+, J2 IN-, J3 TW+, J4 TW-, J5 WF+, J6 WF-

Commit message: Fixed L1 and L2 footprints
Parts:
- turned L2 to 0 degrees
Connections:
- L2 pad 1: Net-(C1-Pad2) -> Net-(C3-Pad1)
- L2 pad 2: Net-(C3-Pad1) -> Net-(C1-Pad2)
Changed lines of the file:
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@@
     (add_net "Net-(J3-Pad1)")
+  )
+  (module Crossover:255-252 (layer F.Cu)
+    (at 73.075001 93.875001)
+    (fp_text reference L2 (at -0.124999 -0.075001 270) (layer F.SilkS)
+      (effects (font (size 1 1) (thickness 0.15)))
+    )
+    (fp_text value 1m1 (at 0 0) (layer F.Fab)
+      (effects (font (size 1 1) (thickness 0.15)))
+    )
+    (fp_line (start -21 -9) (end -21 -21) (layer F.CrtYd) (width 0.12))
+    (fp_line (start -21 21) (end -21 -9) (layer F.CrtYd) (width 0.12))
+    (fp_line (start 21 21) (end -21 21) (layer F.CrtYd) (width 0.12))
+    (fp_line (start 21 -21) (end 21 21) (layer F.CrtYd) (width 0.12))
+    (fp_line (start -21 -21) (end 21 -21) (layer F.CrtYd) (width 0.12))
+    (fp_circle (center 0 0) (end 12.5 0) (layer F.SilkS) (width 0.15))
+    (fp_circle (center 0 0) (end 21 0) (layer F.SilkS) (width 0.15))
+    (pad 2 thru_hole circle (at -7.3 -10.2) (size 2 2) (drill 1.3) (layers *.Cu *.Mask)
+      (net 2 "Net-(C1-Pad2)"))
+    (pad 1 thru_hole circle (at 0 21) (size 2 2) (drill 1.3) (layers *.Cu *.Mask)
+      (net 4 "Net-(C3-Pad1)"))
+  )
+  (module Crossover:255-030 (layer F.Cu)
+    (at 122 65.5)
+    (fp_text reference L1 (at 0 0) (layer F.SilkS)
+      (effects (font (size 1 1) (thickness 0.15)))
+    )
+    (fp_text value 350m (at 0 0.25) (layer F.Fab)
+      (effects (font (size 1 1) (thickness 0.15)))
+    )
+    (fp_line (start -15 -1) (end -15 -15) (layer F.CrtYd) (width 0.12))
+    (fp_line (start -16 -1) (end -15 -1) (layer F.CrtYd) (width 0.12))
+    (fp_line (start -16 1) (end -16 -1) (layer F.CrtYd) (width 0.12))
+    (fp_line (start -15 1) (end -16 1) (layer F.CrtYd) (width 0.12))
+    (fp_line (start -15 15) (end -15 1) (layer F.CrtYd) (width 0.12))
+    (fp_line (start 15 15) (end -15 15) (layer F.CrtYd) (width 0.12))
+    (fp_line (start 15 -15) (end 15 15) (layer F.CrtYd) (width 0.12))
+    (fp_line (start -15 -15) (end 15 -15) (layer F.CrtYd) (width 0.12))
+    (fp_circle (center 0 0) (end 7.5 0.5) (layer F.SilkS) (width 0.15))
+    (fp_circle (center 0 0) (end 15 0) (layer F.SilkS) (width 0.15))
+    (pad 2 thru_hole circle (at 7.5 0) (size 1.8 1.8) (drill 1.1) (layers *.Cu *.Mask)
+      (net 1 "Net-(C1-Pad1)"))
+    (pad 1 thru_hole circle (at -15 0) (size 1.8 1.8) (drill 1.1) (layers *.Cu *.Mask)
+      (net 5 GND))
   )
   (module Crossover:NPTH_3.5mm_antipad_7mm (layer F.Cu)
@@
       (net 5 GND))
     (pad 2 thru_hole circle (at 24.5 0 180) (size 1.7 1.7) (drill 1) (layers *.Cu *.Mask)
-      (net 4 "Net-(C3-Pad1)"))
-  )
-  (module Crossover:255-252 (layer F.Cu)
-    (at 73.075001 93.875001 90)
-    (fp_text reference L2 (at -0.124999 -0.075001 180) (layer F.SilkS)
-      (effects (font (size 1 1) (thickness 0.15)))
-    )
-    (fp_text value 1m1 (at 0 0 90) (layer F.Fab)
-      (effects (font (size 1 1) (thickness 0.15)))
-    )
-    (fp_circle (center 0 0) (end 21 0) (layer F.SilkS) (width 0.15))
-    (fp_circle (center 0 0) (end 12.5 0) (layer F.SilkS) (width 0.15))
-    (fp_line (start -21 -21) (end 21 -21) (layer F.CrtYd) (width 0.12))
-    (fp_line (start 21 -21) (end 21 21) (layer F.CrtYd) (width 0.12))
-    (fp_line (start 21 21) (end -21 21) (layer F.CrtYd) (width 0.12))
-    (fp_line (start -21 21) (end -21 -9) (layer F.CrtYd) (width 0.12))
-    (fp_line (start -21 -9) (end -21 -21) (layer F.CrtYd) (width 0.12))
-    (pad 1 thru_hole circle (at 0 12.5 90) (size 2 2) (drill 1.3) (layers *.Cu *.Mask)
-      (net 2 "Net-(C1-Pad2)"))
-    (pad 2 thru_hole circle (at -20 -10 90) (size 2 2) (drill 1.3) (layers *.Cu *.Mask)
       (net 4 "Net-(C3-Pad1)"))
   )
@@
       (net 5 GND))
   )
-  (module Crossover:255-030 (layer F.Cu)
-    (at 122 65.5)
-    (fp_text reference L1 (at 0 0) (layer F.SilkS)
-      (effects (font (size 1 1) (thickness 0.15)))
-    )
-    (fp_text value 350m (at 0 0.25) (layer F.Fab)
-      (effects (font (size 1 1) (thickness 0.15)))
-    )
-    (fp_circle (center 0 0) (end 15 0) (layer F.SilkS) (width 0.15))
-    (fp_circle (center 0 0) (end 7.5 0.5) (layer F.SilkS) (width 0.15))
-    (fp_line (start -15 -15) (end 15 -15) (layer F.CrtYd) (width 0.12))
-    (fp_line (start 15 -15) (end 15 15) (layer F.CrtYd) (width 0.12))
-    (fp_line (start 15 15) (end -15 15) (layer F.CrtYd) (width 0.12))
-    (fp_line (start -15 15) (end -15 1) (layer F.CrtYd) (width 0.12))
-    (fp_line (start -15 1) (end -16 1) (layer F.CrtYd) (width 0.12))
-    (fp_line (start -16 1) (end -16 -1) (layer F.CrtYd) (width 0.12))
-    (fp_line (start -16 -1) (end -15 -1) (layer F.CrtYd) (width 0.12))
-    (fp_line (start -15 -1) (end -15 -15) (layer F.CrtYd) (width 0.12))
-    (pad 1 thru_hole circle (at -15 0) (size 1.8 1.8) (drill 1.1) (layers *.Cu *.Mask)
-      (net 5 GND))
-    (pad 2 thru_hole circle (at -7.5 0) (size 1.8 1.8) (drill 1.1) (layers *.Cu *.Mask)
-      (net 1 "Net-(C1-Pad1)"))
-  )
   (module Crossover:DNR_10W (layer F.Cu)
     (at 78.560001 67)
@@
       (pts
         (xy 101 55) (xy 101 64) (xy 103 66) (xy 103 89) (xy 110 96)
-        (xy 110 125) (xy 135 125) (xy 135 119) (xy 146 111) (xy 146 91)
-        (xy 136 91) (xy 111 66) (xy 111 54) (xy 102 54)
+        (xy 110 125) (xy 135 125) (xy 135 119) (xy 146 111) (xy 146 92)
+        (xy 134 92) (xy 117 75) (xy 117 62) (xy 109 54) (xy 102 54)
       )
     )
@@
     (polygon
       (pts
-        (xy 95 89) (xy 87 97) (xy 82 97) (xy 72 87) (xy 72 43)
+        (xy 95 89) (xy 87 97) (xy 72 97) (xy 62 87) (xy 62 43)
         (xy 52 43) (xy 52 100) (xy 89 100) (xy 97 92) (xy 100 92)
         (xy 102 94) (xy 105 97) (xy 105 125) (xy 109 125) (xy 109 113)
         (xy 109 96) (xy 102 89)
+      )
+    )
+  )
+  (zone (net 2) (net_name "Net-(C1-Pad2)") (layer B.Cu) (hatch edge 0.508)
+    (connect_pads (clearance 0.508))
+    (min_thickness 0.254)
+    (fill yes (arc_segments 32) (thermal_gap 0.508) (thermal_bridge_width 0.508))
+    (polygon
+      (pts
+        (xy 150 125) (xy 150 43) (xy 63 43) (xy 63 86) (xy 73 96)
+        (xy 87 96) (xy 95 88) (xy 102 88) (xy 102 66) (xy 100 64)
+        (xy 100 55) (xy 102 53) (xy 109 53) (xy 118 62) (xy 130 62)
+        (xy 147 79) (xy 147 111) (xy 136 119) (xy 136 125)
       )
     )
@@
     (polygon
       (pts
-        (xy 112 54) (xy 112 65) (xy 112 66) (xy 136 90) (xy 146 90)
-        (xy 146 79) (xy 121 54)
+        (xy 130 63) (xy 146 79) (xy 146 91) (xy 134 91) (xy 118 75)
+        (xy 118 63)
       )
     )
-  )
-  (zone (net 2) (net_name "Net-(C1-Pad2)") (layer B.Cu) (hatch edge 0.508)
-    (connect_pads (clearance 0.508))
-    (min_thickness 0.254)
-    (fill yes (arc_segments 32) (thermal_gap 0.508) (thermal_bridge_width 0.508))
-    (polygon
-      (pts
-        (xy 150 125) (xy 150 43) (xy 73 43) (xy 73 87) (xy 82 96)
-        (xy 87 96) (xy 95 88) (xy 102 88) (xy 102 66) (xy 100 64)
-        (xy 100 55) (xy 102 53) (xy 121 53) (xy 147 79) (xy 147 111)
-        (xy 136 119) (xy 136 125)
-      )
-    )
