File: crossover/crossover.sch (KiCad schematic (older format))
At the start: 14 parts, among them J1 IN+, J2 IN-, J3 TW+, J4 TW-, J5 WF+, J6 WF-

Commit message: Added footprints
Parts:
- C1: footprint (none) -> Crossover:DMPC-1.5
- C2: footprint (none) -> Crossover:DMPC-2.2
- C3: footprint (none) -> Crossover:DMPC-0.22
- C4: footprint (none) -> Crossover:DMPC-6.8
- J1, J2, J3, J4, J5, J6: footprint (none) -> Crossover:TAB_378005.68
- L1: value 350n -> 350m; footprint (none) -> Crossover:255-030
- L2: value 350n -> 1m1; footprint (none) -> Crossover:255-252
- R1, R2: footprint (none) -> Crossover:DNR_10W
Changed lines of the file:
@@
 EESchema Schematic File Version 4
+LIBS:crossover-cache
 EELAYER 26 0
 EELAYER END
@@
 F 0 "J1" H 4500 2950 50  0000 C CNN
 F 1 "IN+" H 4500 2850 50  0000 C CNN
-F 2 "" H 4350 2900 50  0001 C CNN
+F 2 "Crossover:TAB_378005.68" H 4350 2900 50  0001 C CNN
 F 3 "~" H 4350 2900 50  0001 C CNN
 	1    4350 2900
@@
 F 0 "J2" H 4500 3250 50  0000 C CNN
 F 1 "IN-" H 4500 3150 50  0000 C CNN
-F 2 "" H 4350 3200 50  0001 C CNN
+F 2 "Crossover:TAB_378005.68" H 4350 3200 50  0001 C CNN
 F 3 "~" H 4350 3200 50  0001 C CNN
 	1    4350 3200
@@
 F 0 "C1" V 4848 2900 50  0000 C CNN
 F 1 "1u5" V 4939 2900 50  0000 C CNN
-F 2 "" H 5138 2750 50  0001 C CNN
+F 2 "Crossover:DMPC-1.5" H 5138 2750 50  0001 C CNN
 F 3 "~" H 5100 2900 50  0001 C CNN
 	1    5100 2900
@@
 P 5350 3150
 F 0 "L1" H 5309 3104 50  0000 R CNN
-F 1 "350n" H 5309 3195 50  0000 R CNN
-F 2 "" H 5350 3150 50  0001 C CNN
+F 1 "350m" H 5309 3195 50  0000 R CNN
+F 2 "Crossover:255-030" H 5350 3150 50  0001 C CNN
 F 3 "~" H 5350 3150 50  0001 C CNN
 	1    5350 3150
@@
 F 0 "C2" V 5348 2900 50  0000 C CNN
 F 1 "2u2" V 5439 2900 50  0000 C CNN
-F 2 "" H 5638 2750 50  0001 C CNN
+F 2 "Crossover:DMPC-2.2" H 5638 2750 50  0001 C CNN
 F 3 "~" H 5600 2900 50  0001 C CNN
 	1    5600 2900
@@
 F 0 "R1" V 5693 2900 50  0000 C CNN
 F 1 "6R" V 5784 2900 50  0000 C CNN
-F 2 "" V 5830 2900 50  0001 C CNN
+F 2 "Crossover:DNR_10W" V 5830 2900 50  0001 C CNN
 F 3 "~" H 5900 2900 50  0001 C CNN
 	1    5900 2900
@@
 F 0 "R2" H 6220 3196 50  0000 L CNN
 F 1 "10R" H 6220 3105 50  0000 L CNN
-F 2 "" V 6080 3150 50  0001 C CNN
+F 2 "Crossover:DNR_10W" V 6080 3150 50  0001 C CNN
 F 3 "~" H 6150 3150 50  0001 C CNN
 	1    6150 3150
@@
 F 0 "J3" H 6930 2942 50  0000 L CNN
 F 1 "TW+" H 6930 2851 50  0000 L CNN
-F 2 "" H 6850 2900 50  0001 C CNN
+F 2 "Crossover:TAB_378005.68" H 6850 2900 50  0001 C CNN
 F 3 "~" H 6850 2900 50  0001 C CNN
 	1    6850 2900
@@
 F 0 "J4" H 6930 3242 50  0000 L CNN
 F 1 "TW-" H 6930 3151 50  0000 L CNN
-F 2 "" H 6850 3200 50  0001 C CNN
+F 2 "Crossover:TAB_378005.68" H 6850 3200 50  0001 C CNN
 F 3 "~" H 6850 3200 50  0001 C CNN
 	1    6850 3200
@@
 F 0 "J5" H 6929 4042 50  0000 L CNN
 F 1 "WF+" H 6929 3951 50  0000 L CNN
-F 2 "" H 6850 4000 50  0001 C CNN
+F 2 "Crossover:TAB_378005.68" H 6850 4000 50  0001 C CNN
 F 3 "~" H 6850 4000 50  0001 C CNN
 	1    6850 4000
@@
 F 0 "J6" H 6929 4342 50  0000 L CNN
 F 1 "WF-" H 6929 4251 50  0000 L CNN
-F 2 "" H 6850 4300 50  0001 C CNN
+F 2 "Crossover:TAB_378005.68" H 6850 4300 50  0001 C CNN
 F 3 "~" H 6850 4300 50  0001 C CNN
 	1    6850 4300
@@
 F 0 "C3" V 5248 3900 50  0000 C CNN
 F 1 "220n" V 5339 3900 50  0000 C CNN
-F 2 "" H 5538 3750 50  0001 C CNN
+F 2 "Crossover:DMPC-0.22" H 5538 3750 50  0001 C CNN
 F 3 "~" H 5500 3900 50  0001 C CNN
 	1    5500 3900
@@
 P 5500 4100
 F 0 "L2" V 5450 4100 50  0000 C CNN
-F 1 "350n" V 5350 4100 50  0000 C CNN
-F 2 "" H 5500 4100 50  0001 C CNN
+F 1 "1m1" V 5350 4100 50  0000 C CNN
+F 2 "Crossover:255-252" H 5500 4100 50  0001 C CNN
 F 3 "~" H 5500 4100 50  0001 C CNN
 	1    5500 4100
@@
 F 0 "C4" H 5835 4204 50  0000 R CNN
 F 1 "6u8" H 5835 4295 50  0000 R CNN
-F 2 "" H 5988 4100 50  0001 C CNN
+F 2 "Crossover:DMPC-6.8" H 5988 4100 50  0001 C CNN
 F 3 "~" H 5950 4250 50  0001 C CNN
 	1    5950 4250

Commit message: Associated footprints
Parts:
- added NPTH1, NPTH2, NPTH3, NPTH4: 3.5mm, Crossover:NPTH_3.5mm_antipad_7mm, symbol Mechanical:MountingHole
Changed lines of the file:
@@
 EESchema Schematic File Version 4
 LIBS:crossover-cache
-EELAYER 26 0
+EELAYER 29 0
 EELAYER END
 $Descr A4 11693 8268
@@
 Text Notes 7200 4200 0    50   ~ 0
 Woofer: HiVi B4N
+$Comp
+L Mechanical:MountingHole NPTH1
+U 1 1 5D34B1E5
+P 750 6900
+F 0 "NPTH1" H 850 6946 50  0000 L CNN
+F 1 "3.5mm" H 850 6855 50  0000 L CNN
+F 2 "Crossover:NPTH_3.5mm_antipad_7mm" H 750 6900 50  0001 C CNN
+F 3 "~" H 750 6900 50  0001 C CNN
+	1    750  6900
+	1    0    0    -1
+$EndComp
+$Comp
+L Mechanical:MountingHole NPTH2
+U 1 1 5D34BA53
+P 750 7100
+F 0 "NPTH2" H 850 7146 50  0000 L CNN
+F 1 "3.5mm" H 850 7055 50  0000 L CNN
+F 2 "Crossover:NPTH_3.5mm_antipad_7mm" H 750 7100 50  0001 C CNN
+F 3 "~" H 750 7100 50  0001 C CNN
+	1    750  7100
+	1    0    0    -1
+$EndComp
+$Comp
+L Mechanical:MountingHole NPTH3
+U 1 1 5D34BB19
+P 750 7300
+F 0 "NPTH3" H 850 7346 50  0000 L CNN
+F 1 "3.5mm" H 850 7255 50  0000 L CNN
+F 2 "Crossover:NPTH_3.5mm_antipad_7mm" H 750 7300 50  0001 C CNN
+F 3 "~" H 750 7300 50  0001 C CNN
+	1    750  7300
+	1    0    0    -1
+$EndComp
+$Comp
+L Mechanical:MountingHole NPTH4
+U 1 1 5D34BBDF
+P 750 7500
+F 0 "NPTH4" H 850 7546 50  0000 L CNN
+F 1 "3.5mm" H 850 7455 50  0000 L CNN
+F 2 "Crossover:NPTH_3.5mm_antipad_7mm" H 750 7500 50  0001 C CNN
+F 3 "~" H 750 7500 50  0001 C CNN
+	1    750  7500
+	1    0    0    -1
+$EndComp
 $EndSCHEMATC

Commit message: Fixed L1 and L2 footprints
Connections:
- net at C1.2, C3.2, J1.1 (Pin_1): now also L2.2; no longer L2.1
- net at C3.1, C4.2, J5.1 (Pin_1): now also L2.1; no longer L2.2
Other:
- moved on the sheet: L2
Changed lines of the file:
@@
 U 1 1 5D2A36E4
 P 5500 4100
-F 0 "L2" V 5450 4100 50  0000 C CNN
-F 1 "1m1" V 5350 4100 50  0000 C CNN
+F 0 "L2" V 5600 4100 50  0000 C CNN
+F 1 "1m1" V 5700 4100 50  0000 C CNN
 F 2 "Crossover:255-252" H 5500 4100 50  0001 C CNN
 F 3 "~" H 5500 4100 50  0001 C CNN
 	1    5500 4100
-	0    -1   -1   0
+	0    1    1    0
 $EndComp
 $Comp
